File: Schematics/MainBoard/MainBoard.sch (KiCad schematic (older format))
At the start: 0 parts

Commit message: Erste Schritte zu einem Funktionalen Schaltplan.
Parts:
- added BT1: Battery, symbol Battery
- added C1: CP, symbol CP
- added C2, C3: C, symbol C
- added C4: C_Small, symbol C_Small
- added D1: D, symbol D
- added D2: LED, symbol LED
- added D3: LED_RCBG, symbol LED_RCBG
- added IC1: ATMEGA32-P, Housings_DIP:DIP-40_W25.4mm, symbol ATMEGA32-P
- added R1, R2, R3, R4, R5, R? (x2): R, symbol R
- added SW1: SW_PUSH, symbol SW_PUSH
- added U1: 7805, symbol 7805
- added Y1: Crystal, symbol Crystal
Connections:
- new net: C2.1, IC1.12 (XTAL2), Y1.1
- new net: C3.1, IC1.13 (XTAL1), Y1.2
- new net: IC1.9 (~RESET), R2.2
- new net: BT1.1, D1.2 (A)
- new net: D2.1 (K), R1.1
- new net: D3.1 (RED_ANODE), R5.1
- new net: D3.3 (BLUE_ANODE), R3.1
- new net: D3.4 (GREEN_ANODE), R4.1
- new net +12V: D1.1 (K), R?.1, U1.VI
- new net +5V: C1.1, C4.1, D2.2 (A), IC1.10 (VCC), IC1.30 (AVCC), IC1.32 (AREF), R2.1, U1.VO
- new net BTN: IC1.5 ((~SS~)PB4), SW1.1
- new net GND: BT1.2, C1.2, C2.2, C3.2, C4.2, D3.2 (COMMON_CATHODE), IC1.11 (GND), IC1.31 (AGND), R1.2, R?.2, SW1.2, U1.GND
- new net MISO: IC1.7 ((MISO)PB6), R4.2
- new net MOSI: IC1.6 ((MOSI)PB5), R3.2
- new net PWMES: IC1.33 ((ADC7)PA7), R?.1, R?.2
- new net SCK: IC1.8 ((SCK)PB7), R5.2
- new net SCL: IC1.22 ((SCL)PC0)
- new net SDA: IC1.23 ((SDA)PC1)
- new net SENS0: IC1.40 ((ADC0)PA0)
- new net SENS1: IC1.39 ((ADC1)PA1)
- new net SENS2: IC1.38 ((ADC2)PA2)
- new net SENS3: IC1.37 ((ADC3)PA3)
- new net SENS4: IC1.36 ((ADC4)PA4)
- new net SENS5: IC1.35 ((ADC5)PA5)
- new net SENS6: IC1.34 ((ADC6)PA6)
- new net STEP0: IC1.1 ((T0/XCK)PB0)
- new net STEP1: IC1.2 ((T1)PB1)
- new net STEPD: IC1.3 ((AIN0/INT2)PB2)
Other:
- note added: "Power systems\n"
- note added: "User Interface\n"

Commit message: Schaltkreise noch ein wenig verfeinert.
Parts:
- added P1, P2, P3, P4, P5, P6, P7: CONN_01X03, symbol CONN_01X03
- added P8: CONN_01X07, symbol CONN_01X07
- gave numbers to parts that had none: 2
Connections:
- net +12V: now also P8.6 (P6)
- net +5V: now also P1.2 (P2), P2.2 (P2), P3.2 (P2), P4.2 (P2), P5.2 (P2), P6.2 (P2), P7.2 (P2), P8.5 (P5)
- net GND: now also P1.3 (P3), P2.3 (P3), P3.3 (P3), P4.3 (P3), P5.3 (P3), P6.3 (P3), P7.3 (P3), P8.7 (P7)
- net SENS0: now also P1.1 (P1)
- net SENS1: now also P2.1 (P1)
- net SENS2: now also P3.1 (P1)
- net SENS3: now also P4.1 (P1)
- net SENS4: now also P5.1 (P1)
- net SENS5: now also P6.1 (P1)
- net SENS6: now also P7.1 (P1)
- net STEP0: now also P8.4 (P4)
- net STEP1: now also P8.3 (P3)
- net STEPD: now also P8.2 (P2)
- net STEPE: now reaches IC1.4 ((AIN1/OC0)PB3)
- net STEPE: now also P8.1 (P1)

Commit message: Schaltplan mit Beschreibungen erweitert und SPI angelegt.
Parts:
- added SPI1: CONN_02X03, symbol CONN_02X03
- C2, C3: value C -> 56pF
- R1, R3, R4, R5: value R -> 1kΩ
- R2: value R -> 5kΩ
- R6: value R -> 4.7kΩ
- R7: value R -> 2.6kΩ
- Y1: value Crystal -> 16MHz
Connections:
- net +5V: now also SPI1.2 (P2)
- net GND: now also SPI1.6 (P6)
- net MISO: now also SPI1.1 (P1)
- net MOSI: now also SPI1.4 (P4)
- net SCK: now also SPI1.3 (P3)
- new net RST: SPI1.5 (P5)
Other:
- note added: "Analog sensor pins"
- note added: "Analog sensor pins\n"
- note added: "Battery measurement\n"
- note added: "I2C Con\n"
- note added: "Programming \n interface"
- note added: "SPI & User interfacing\n"
- note added: "Stepper connections"
- note added: "Stepper driver connection"

Commit message: Werte für den Kondensator hinzugefügt.
Parts:
- C1: value CP -> 220uF
Other:
- moved on the sheet: C1
Changed lines of the file:
@@
 $EndComp
 Wire Wire Line
-	9400 5700 9500 5700
+	9400 5700 9450 5700
+Wire Wire Line
+	9450 5700 9500 5700
 $Comp
 L GND #PWR19
@@
 $EndComp
 Wire Wire Line
-	9000 6000 9000 6100
+	9000 6000 9000 6050
+Wire Wire Line
+	9000 6050 9000 6100
 $Comp
 L CP C1
 U 1 1 57B975BF
-P 9450 5900
-F 0 "C1" H 9475 6000 50  0000 L CNN
-F 1 "CP" H 9475 5800 50  0000 L CNN
-F 2 "" H 9488 5750 50  0000 C CNN
-F 3 "" H 9450 5900 50  0000 C CNN
-	1    9450 5900
-	1    0    0    -1
-$EndComp
-Wire Wire Line
-	9450 5750 9450 5700
+P 9400 5900
+F 0 "C1" H 9425 6000 50  0000 L CNN
+F 1 "220uF" H 9425 5800 50  0000 L CNN
+F 2 "" H 9438 5750 50  0000 C CNN
+F 3 "" H 9400 5900 50  0000 C CNN
+	1    9400 5900
+	1    0    0    -1
+$EndComp
+Wire Wire Line
+	9400 5750 9450 5700
 Connection ~ 9450 5700
 Wire Wire Line
-	9450 6050 9000 6050
+	9400 6050 9000 6050
 Connection ~ 9000 6050
 $Comp
@@
 $EndComp
 Wire Wire Line
-	3750 6000 3750 6200
+	3750 6000 3750 6100
+Wire Wire Line
+	3750 6100 3750 6200
 Wire Wire Line
 	3750 6100 3850 6100
@@
 $EndComp
 Wire Wire Line
-	3650 1850 3650 2000
+	3650 1850 3650 1900
+Wire Wire Line
+	3650 1900 3650 2000
 Wire Wire Line
 	3650 1900 3950 1900
@@
 $EndComp
 Wire Wire Line
-	2550 3500 2800 3500
+	2550 3500 2650 3500
+Wire Wire Line
+	2650 3500 2800 3500
 $Comp
 L C_Small C4
@@
 	2550 3050 2550 3100
 Wire Wire Line
-	2300 3100 2800 3100
+	2300 3100 2550 3100
+Wire Wire Line
+	2550 3100 2800 3100
 Wire Wire Line
 	2550 2750 2550 2700
 Wire Wire Line
-	2300 2700 2800 2700
+	2300 2700 2550 2700
+Wire Wire Line
+	2550 2700 2800 2700
 $Comp
 L C C2
@@
 $EndComp
 Wire Wire Line
-	1900 2700 1900 3250
+	1900 2700 1900 3100
+Wire Wire Line
+	1900 3100 1900 3250
 Wire Wire Line
 	1900 3100 2000 3100
@@
 $EndComp
 Wire Wire Line
-	9800 3700 9800 4550
+	9800 3700 9800 4350
+Wire Wire Line
+	9800 4350 9800 4550
 Connection ~ 9800 4350
 $Comp
@@
 	9100 3900 9200 3900
 Wire Bus Line
-	5200 1450 5200 5650
+	5200 1450 5200 2400
+Wire Bus Line
+	5200 2400 5200 2500
+Wire Bus Line
+	5200 2500 5200 2600
+Wire Bus Line
+	5200 2600 5200 2700
+Wire Bus Line
+	5200 2700 5200 2800
+Wire Bus Line
+	5200 2800 5200 2900
+Wire Bus Line
+	5200 2900 5200 3000
+Wire Bus Line
+	5200 3000 5200 3100
+Wire Bus Line
+	5200 3100 5200 3300
+Wire Bus Line
+	5200 3300 5200 3400
+Wire Bus Line
+	5200 3400 5200 3500
+Wire Bus Line
+	5200 3500 5200 3600
+Wire Bus Line
+	5200 3600 5200 3700
+Wire Bus Line
+	5200 3700 5200 3800
+Wire Bus Line
+	5200 3800 5200 3900
+Wire Bus Line
+	5200 3900 5200 4000
+Wire Bus Line
+	5200 4000 5200 4200
+Wire Bus Line
+	5200 4200 5200 4300
+Wire Bus Line
+	5200 4300 5200 5650
 Entry Wire Line
 	5100 4100 5200 4200
@@
 $EndComp
 Wire Wire Line
-	7900 5700 7900 5800
+	7900 5700 7900 5750
+Wire Wire Line
+	7900 5750 7900 5800
 Wire Wire Line
 	7900 5750 7500 5750
@@
 	7350 4950 8450 4950
 Wire Bus Line
-	8450 4950 8450 3600
+	8450 4950 8450 4450
+Wire Bus Line
+	8450 4450 8450 4000
+Wire Bus Line
+	8450 4000 8450 3800
+Wire Bus Line
+	8450 3800 8450 3600
 Entry Wire Line
 	8450 4450 8550 4350
@@
 	7900 2000 7900 2150
 Wire Wire Line
-	7900 2150 10600 2150
+	7900 2150 8000 2150
+Wire Wire Line
+	8000 2150 8350 2150
+Wire Wire Line
+	8350 2150 8800 2150
+Wire Wire Line
+	8800 2150 9250 2150
+Wire Wire Line
+	9250 2150 9700 2150
+Wire Wire Line
+	9700 2150 10150 2150
+Wire Wire Line
+	10150 2150 10600 2150
 Wire Wire Line
 	10150 2150 10150 2000
@@
 Connection ~ 8350 2150
 Wire Wire Line
-	7750 2200 10550 2200
+	7750 2200 7850 2200
+Wire Wire Line
+	7850 2200 8300 2200
+Wire Wire Line
+	8300 2200 8750 2200
+Wire Wire Line
+	8750 2200 9200 2200
+Wire Wire Line
+	9200 2200 9650 2200
+Wire Wire Line
+	9650 2200 10100 2200
+Wire Wire Line
+	10100 2200 10550 2200
 Wire Wire Line
 	7900 1900 7850 1900
@@
 	10500 1450 10600 1550
 Wire Bus Line
-	5200 1450 10500 1450
+	5200 1450 7700 1450
+Wire Bus Line
+	7700 1450 7800 1450
+Wire Bus Line
+	7800 1450 7900 1450
+Wire Bus Line
+	7900 1450 8000 1450
+Wire Bus Line
+	8000 1450 8250 1450
+Wire Bus Line
+	8250 1450 8700 1450
+Wire Bus Line
+	8700 1450 9150 1450
+Wire Bus Line
+	9150 1450 9600 1450
+Wire Bus Line
+	9600 1450 10050 1450
+Wire Bus Line
+	10050 1450 10500 1450
 $Comp
 L GND #PWR15
@@
 	6450 800  6550 900
 Wire Bus Line
-	5450 800  5450 1450
+	5450 800  5450 900
+Wire Bus Line
+	5450 900  5450 1000
+Wire Bus Line
+	5450 1000 5450 1450
 Wire Bus Line
 	6550 900  6550 900

Commit message: Überspannungsdiode, I2C, Sicherung hinzugefügt.
Parts:
- added D?: ZENER, symbol ZENER
- added F1: F_Small, symbol F_Small
- added I2C1: CONN_02X02, symbol CONN_02X02
Connections:
- net +5V: now also D?.1 (K), F1.2, I2C1.3 (P3); no longer C1.1, U1.VO
- net GND: now also D?.2 (A), I2C1.4 (P4)
- net SCL: now also I2C1.2 (P2)
- net SDA: now also I2C1.1 (P1)
- new net: C1.1, F1.1, U1.VO
Other:
- note added: "I2C \n Coms\n"
- moved on the sheet: BT1, C1, D1, U1

Commit message: Anfang der Verlegung des PSU-Systemes auf separaten Chip.
Parts:
- removed BT1: Battery, symbol Battery
- removed C1: 220uF, symbol CP
- removed D1: D, symbol D
- removed D2: LED, symbol LED
- removed D?: ZENER, symbol ZENER
- removed F1: F_Small, symbol F_Small
- removed R1: 1kΩ, symbol R
- removed R6: 4.7kΩ, symbol R
- removed R7: 2.6kΩ, symbol R
- removed U1: 7805, symbol 7805
Other:
- note removed: "Power systems\n"
- moved on the sheet: C2, C3, C4, IC1, R2, Y1

Commit message: Beendung des Umänderns des Platinen-Designs. Das neue System beinhaltet nun: - Alle für den Roboter relevanten Bauteile (inclusive A4988 Treiber) - Erweiterte Dokumentation des Schaltkreises - Ein separater Schaltplan rein für die Strom-Elektronik & Sicherheit (gemäß der Aufspaltung auf zwei separate Hardware-Platinen)
Parts:
- removed P8: CONN_01X07, symbol CONN_01X07
Connections:
- net PWMES renamed VSens
Other:
- note removed: "Stepper driver connection"
Changed lines of the file:
@@
 $EndComp
 $Comp
-L GND #PWR16
+L GND #PWR18
 U 1 1 57B9F26B
 P 9800 4550
-F 0 "#PWR16" H 9800 4300 50  0001 C CNN
+F 0 "#PWR18" H 9800 4300 50  0001 C CNN
 F 1 "GND" H 9800 4400 50  0000 C CNN
 F 2 "" H 9800 4550 50  0000 C CNN
@@
 SENS6
 Text Label 3550 1850 0    60   ~ 0
-PWMES
+VSens
 Wire Wire Line
 	3550 2050 3850 2050
@@
 	10150 1550 10150 1800
 $Comp
-L GND #PWR12
+L GND #PWR14
 U 1 1 57BB6AC8
 P 8000 2300
-F 0 "#PWR12" H 8000 2050 50  0001 C CNN
+F 0 "#PWR14" H 8000 2050 50  0001 C CNN
 F 1 "GND" H 8000 2150 50  0000 C CNN
 F 2 "" H 8000 2300 50  0000 C CNN
@@
 Connection ~ 8000 2150
 $Comp
-L +5V #PWR11
+L +5V #PWR13
 U 1 1 57BB6CE4
 P 7750 2200
-F 0 "#PWR11" H 7750 2050 50  0001 C CNN
+F 0 "#PWR13" H 7750 2050 50  0001 C CNN
 F 1 "+5V" H 7750 2340 50  0000 C CNN
 F 2 "" H 7750 2200 50  0000 C CNN
@@
 Wire Bus Line
 	10050 1450 10500 1450
-$Comp
-L GND #PWR13
-U 1 1 57BBF5F4
-P 8400 1200
-F 0 "#PWR13" H 8400 950 50  0001 C CNN
-F 1 "GND" H 8400 1050 50  0000 C CNN
-F 2 "" H 8400 1200 50  0000 C CNN
-F 3 "" H 8400 1200 50  0000 C CNN
-	1    8400 1200
-	1    0    0    -1
-$EndComp
-Wire Wire Line
-	8400 1200 8400 950
-Wire Wire Line
-	8300 950  8300 1000
-Wire Wire Line
-	8300 1000 8550 1000
-Wire Wire Line
-	8550 1000 8550 950
-$Comp
-L +12V #PWR14
-U 1 1 57BBFAFB
-P 8550 950
-F 0 "#PWR14" H 8550 800 50  0001 C CNN
-F 1 "+12V" H 8550 1090 50  0000 C CNN
-F 2 "" H 8550 950 50  0000 C CNN
-F 3 "" H 8550 950 50  0000 C CNN
-	1    8550 950
-	1    0    0    -1
-$EndComp
-$Comp
-L +5V #PWR15
-U 1 1 57BBFB45
-P 8800 950
-F 0 "#PWR15" H 8800 800 50  0001 C CNN
-F 1 "+5V" H 8800 1090 50  0000 C CNN
-F 2 "" H 8800 950 50  0000 C CNN
-F 3 "" H 8800 950 50  0000 C CNN
-	1    8800 950
-	1    0    0    -1
-$EndComp
-Wire Wire Line
-	8800 950  8800 1050
-Wire Wire Line
-	8800 1050 8200 1050
-Wire Wire Line
-	8200 1050 8200 950
 Wire Wire Line
 	3550 2350 3850 2350
@@
 Text Label 3550 2350 0    60   ~ 0
 STEPE
-$Comp
-L CONN_01X07 P8
-U 1 1 57BC11F0
-P 8100 750
-F 0 "P8" H 8100 1150 50  0000 C CNN
-F 1 "CONN_01X07" V 8200 750 50  0000 C CNN
-F 2 "" H 8100 750 50  0000 C CNN
-F 3 "" H 8100 750 50  0000 C CNN
-	1    8100 750
-	0    -1   -1   0
-$EndComp
-Wire Wire Line
-	8100 950  8100 1350
-Wire Wire Line
-	8000 950  8000 1350
-Wire Wire Line
-	7900 950  7900 1350
-Wire Wire Line
-	7800 950  7800 1350
-Text Label 8100 1200 1    60   ~ 0
-STEP0
-Text Label 8000 1200 1    60   ~ 0
-STEP1
-Text Label 7900 1200 1    60   ~ 0
-STEPD
-Text Label 7800 1200 1    60   ~ 0
-STEPE
-Entry Wire Line
-	7700 1450 7800 1350
-Entry Wire Line
-	7800 1450 7900 1350
-Entry Wire Line
-	7900 1450 8000 1350
-Entry Wire Line
-	8000 1450 8100 1350
 Wire Notes Line
 	3550 1050 4000 1050
@@
 Wire Notes Line
 	4000 3050 3550 3050
-Text Notes 4050 1450 0    60   ~ 0
+Text Notes 4050 1650 0    60   ~ 0
 Analog sensor pins\n
 Text Notes 4050 1950 0    60   ~ 0
@@
 	6350 700  6350 650
 $Comp
-L +5V #PWR9
+L +5V #PWR11
 U 1 1 57BC21BF
 P 6350 650
-F 0 "#PWR9" H 6350 500 50  0001 C CNN
+F 0 "#PWR11" H 6350 500 50  0001 C CNN
 F 1 "+5V" H 6350 790 50  0000 C CNN
 F 2 "" H 6350 650 50  0000 C CNN
@@
 $EndComp
 $Comp
-L GND #PWR10
+L GND #PWR12
 U 1 1 57BC2537
 P 6350 900
-F 0 "#PWR10" H 6350 650 50  0001 C CNN
+F 0 "#PWR12" H 6350 650 50  0001 C CNN
 F 1 "GND" H 6350 750 50  0000 C CNN
 F 2 "" H 6350 900 50  0000 C CNN
@@
 Text Notes 7650 2600 0    60   ~ 0
 Analog sensor pins
-Wire Notes Line
-	7650 1400 8900 1400
-Wire Notes Line
-	8900 1400 8900 600
-Wire Notes Line
-	8900 600  7650 600
-Wire Notes Line
-	7650 600  7650 1400
-Text Notes 7650 600  0    60   ~ 0
-Stepper driver connection
 $Comp
 L CONN_02X02 I2C1
@@
 $EndComp
 $Comp
-L GND #PWR8
+L GND #PWR10
 U 1 1 57DB64EF
 P 5100 1000
-F 0 "#PWR8" H 5100 750 50  0001 C CNN
+F 0 "#PWR10" H 5100 750 50  0001 C CNN
 F 1 "GND" H 5100 850 50  0000 C CNN
 F 2 "" H 5100 1000 50  0000 C CNN
@@
 	5100 850  5100 1000
 $Comp
-L +5V #PWR7
+L +5V #PWR9
 U 1 1 57DB67FE
 P 4400 1050
-F 0 "#PWR7" H 4400 900 50  0001 C CNN
+F 0 "#PWR9" H 4400 900 50  0001 C CNN
 F 1 "+5V" H 4400 1190 50  0000 C CNN
 F 2 "" H 4400 1050 50  0000 C CNN
@@
 Wire Bus Line
 	3950 3050 3950 3150
+Wire Bus Line
+	3950 3150 3950 5900
+Wire Bus Line
+	3950 5900 3950 6100
+Wire Bus Line
+	3950 6100 3950 6200
+Wire Bus Line
+	3950 6200 3950 6300
+Wire Bus Line
+	3950 6300 3950 6400
 Wire Bus Line
 	8450 3300 8450 3600
@@
 F3 "+5V" I R 3450 5900 60
 F4 "VSens" I R 3450 6000 60
+F5 "STEP0" I R 3450 6500 60
+F6 "STEP1" I R 3450 6400 60
+F7 "STEPD" I R 3450 6300 60
+F8 "STEPE" I R 3450 6200 60
 $EndSheet
+$Comp
+L +5V #PWR7
+U 1 1 57E538BF
+P 3600 5800
+F 0 "#PWR7" H 3600 5650 50  0001 C CNN
+F 1 "+5V" H 3600 5940 50  0000 C CNN
+F 2 "" H 3600 5800 50  0000 C CNN
+F 3 "" H 3600 5800 50  0000 C CNN
+	1    3600 5800
+	1    0    0    -1
+$EndComp
+Wire Wire Line
+	3450 5900 3600 5900
+Wire Wire Line
+	3600 5900 3600 5800
+$Comp
+L GND #PWR8
+U 1 1 57E53B40
+P 3600 6850
+F 0 "#PWR8" H 3600 6600 50  0001 C CNN
+F 1 "GND" H 3600 6700 50  0000 C CNN
+F 2 "" H 3600 6850 50  0000 C CNN
+F 3 "" H 3600 6850 50  0000 C CNN
+	1    3600 6850
+	1    0    0    -1
+$EndComp
+Wire Wire Line
+	3450 6750 3600 6750
+Wire Wire Line
+	3600 6750 3600 6850
+Wire Wire Line
+	3450 6500 3850 6500
+Wire Wire Line
+	3450 6400 3850 6400
+Wire Wire Line
+	3450 6300 3850 6300
+Wire Wire Line
+	3450 6200 3850 6200
+Entry Wire Line
+	3850 6200 3950 6100
+Entry Wire Line
+	3850 6300 3950 6200
+Entry Wire Line
+	3850 6400 3950 6300
+Entry Wire Line
+	3850 6500 3950 6400
+Text Label 3500 6200 0    60   ~ 0
+STEPE
+Text Label 3500 6300 0    60   ~ 0
+STEPD
+Text Label 3500 6400 0    60   ~ 0
+STEP1
+Text Label 3500 6500 0    60   ~ 0
+STEP0
+Wire Wire Line
+	3450 6000 3850 6000
+Text Label 3500 6000 0    60   ~ 0
+VSens
+Entry Wire Line
+	3850 6000 3950 5900
 $EndSCHEMATC

Commit message: Footprints der Teile hinzugefügt.
Parts:
- C2, C3: footprint (none) -> Capacitors_ThroughHole:C_Disc_D3_P2.5
- C4: footprint (none) -> Capacitors_ThroughHole:C_Radial_D10_L16_P5
- D3: footprint (none) -> LEDs:LED-RGB-5MM_Common_Cathode
- I2C1: footprint (none) -> Pin_Headers:Pin_Header_Straight_2x02
- P1, P2, P3, P4, P5, P6, P7: footprint (none) -> Pin_Headers:Pin_Header_Straight_1x02
- R2, R3, R4, R5: footprint (none) -> Discret:R1
- SPI1: footprint (none) -> Pin_Headers:Pin_Header_Angled_2x03
- SW1: footprint (none) -> Buttons_Switches_ThroughHole:SW_PUSH_6mm
